File: kicad/instrumento/power.kicad_sch (KiCad schematic)
At the start: 6 parts

Commit message: Audio output
Connections:
- net GND: now also BMS1. (V-)
- new net: BMS1. (V-), SD1. (OUT-), SU1. (GND)
Other:
- moved on the sheet: SD1, SU1
